File: picotronix.kicad_sch (KiCad schematic)
At the start: 20 parts

Commit message: finish rev 1
Parts:
- removed D? (x3): LED, symbol Device:LED
- removed J?: Conn_02x04_Top_Bottom, symbol Connector_Generic:Conn_02x04_Top_Bottom
- removed R? (x2): R_US, symbol Device:R_US
- removed SW?: RotaryEncoder_Switch, symbol Device:RotaryEncoder_Switch
- added C1, C2, C5: 0.1u, Capacitor_SMD:C_0603_1608Metric_Pad1.08x0.95mm_HandSolder, symbol Device:C_Small
- added C6: 1u, Capacitor_SMD:C_0603_1608Metric_Pad1.08x0.95mm_HandSolder, symbol Device:C_Small
- added H1, H2, H3, H4: MountingHole, MountingHole:MountingHole_3.2mm_M3, symbol Mechanical:MountingHole
- added J1, J2: Conn_02x04_Odd_Even, Connector_PinSocket_2.54mm:PinSocket_2x04_P2.54mm_Vertical, symbol Connector_Generic:Conn_02x04_Odd_Even
- added J3: DEBUG, Connector_PinHeader_2.54mm:PinHeader_1x03_P2.54mm_Vertical, symbol Connector:Conn_01x03_Male
- added JP1: filter_bypass, Jumper:SolderJumper-2_P1.3mm_Open_Pad1.0x1.5mm, symbol Jumper:SolderJumper_2_Open
- added R1: 10k, Resistor_SMD:R_0603_1608Metric_Pad0.98x0.95mm_HandSolder, symbol Device:R_US
- added RV1: Z Trim, Potentiometer_SMD:Potentiometer_Bourns_TC33X_Vertical, symbol Device:R_Potentiometer_Trim_US
- added RV2: X Trim, Potentiometer_SMD:Potentiometer_Bourns_TC33X_Vertical, symbol Device:R_Potentiometer_Trim_US
- added RV3: Y Trim, Potentiometer_SMD:Potentiometer_Bourns_TC33X_Vertical, symbol Device:R_Potentiometer_Trim_US
- C3, C4: renamed from C?; footprint (none) -> Capacitor_SMD:C_0603_1608Metric_Pad1.08x0.95mm_HandSolder
- J4: renamed from J?; footprint (none) -> Connector_Dsub:DSUB-25_Male_Horizontal_P2.77x2.54mm_EdgePinOffset9.40mm
- R2, R3: renamed from R?; footprint (none) -> Resistor_SMD:R_0603_1608Metric_Pad0.98x0.95mm_HandSolder
- U1: renamed from U?; footprint RPi_Pico:RPi_Pico_SMD_TH -> picotronix:RPi_Pico_SMD_TH
- U4: renamed from U?; footprint (none) -> Package_SO:SOIC-14_3.9x8.7mm_P1.27mm
- gave numbers to parts that had none: 2
Connections:
- net +3V3: now also C1.1, J1.8 (Pin_8), J2.8 (Pin_8), R1.2; no longer U2.8 (OE)
- net +5V: now also C2.1, C5.1, C6.1
- net GND: now also C1.2, C2.2, C5.2, C6.2, J1.1 (Pin_1), J2.1 (Pin_1), J3.3 (Pin_3), RV1.3, RV2.3, RV3.3
- net z_pwm: now also U1.21 (GPIO16), RV1.1; no longer U1.34 (GPIO28_ADC2)
- net at R2.1: now also JP1.1 (A), RV1.2
- net at U3.1 (V_{OUT}A): now also RV2.1; no longer U4.3 (+)
- net gpio0: now reaches U1.1 (GPIO0)
- net gpio0: now also J1.2 (Pin_2)
- net gpio7: now reaches U1.10 (GPIO7)
- net gpio7: now also J2.3 (Pin_3)
- net gpio8: now reaches U1.11 (GPIO8)
- net gpio8: now also J2.4 (Pin_4)
- net gpio9: now reaches U1.12 (GPIO9)
- net gpio9: now also J2.5 (Pin_5)
- net gpio10: now reaches U1.14 (GPIO10)
- net gpio10: now also J2.6 (Pin_6)
- net gpio11: now reaches U1.15 (GPIO11)
- net gpio11: now also J2.7 (Pin_7)
- net gpio1: now reaches U1.2 (GPIO1)
- net gpio1: now also J1.3 (Pin_3)
- net ~{CS}: now reaches U1.22 (GPIO17)
- net ~{CS}: now also U3.6 (~{SYNC})
- net SCLK: now reaches U1.24 (GPIO18)
- net SCLK: now also U3.7 (SCLK)
- net SDO: now reaches U1.25 (GPIO19)
- net SDO: now also U3.8 (D_{IN})
- net XY_FLUSH: now reaches U1.26 (GPIO20)
- net XY_FLUSH: now also U3.4 (~{LDAC})
- net erase_l: now reaches U1.27 (GPIO21)
- net erase_l: now also U2.5 (A4)
- net non_store_l: now reaches U1.29 (GPIO22)
- net non_store_l: now also U2.4 (A3)
- net erase_interval_l: now reaches U1.31 (GPIO26_ADC0)
- net erase_interval_l: now also U2.3 (A2)
- net var_bright_l: now reaches U1.32 (GPIO27_ADC1)
- net var_bright_l: now also U2.2 (A1)
- net gpio2: now reaches U1.4 (GPIO2)
- net gpio2: now also J1.4 (Pin_4)
- net at U1.41 (SWCLK): now also J3.2 (Pin_2)
- net at U1.43 (SWDIO): now also J3.1 (Pin_1)
- net gpio3: now reaches U1.5 (GPIO3)
- net gpio3: now also J1.5 (Pin_5)
- net gpio4: now reaches U1.6 (GPIO4)
- net gpio4: now also J1.6 (Pin_6)
- net gpio5: now reaches U1.7 (GPIO5)
- net gpio5: now also J1.7 (Pin_7)
- net gpio6: now reaches U1.9 (GPIO6)
- net gpio6: now also J2.2 (Pin_2)
- net at C3.2, R3.2, U4.10 (+): now also JP1.2 (B)
- net at U3.2 (V_{OUT}B): now also RV3.1; no longer U4.5 (+)
- new net: RV2.2, U4.3 (+)
- new net: R1.1, U2.8 (OE)
- new net: RV3.2, U4.5 (+)
- no-connect marks 17 -> 20
Other:
- note added: "expansion ports are designed to be ESP-01 compatible"
- note added: "trim pots allow for ranging from 0-3.3v maximum."
- moved on the sheet: C3, R3, U3, U4E
