File: pcb/picotronix.kicad_sch (KiCad schematic)
At the start: 46 parts, among them J1 AudioJack3_Ground, J2 DEBUG, J3 DB25_Male, J4 ESP-01 Connector, SW1 RESET, SW2 BTN0, SW3 BTN1, U1 PCM1808, U2 LSF0204DPWR, U3 Pico, U4 ADA4891-3, U5 AD5663R, U6 W25Q128JVS

Commit message: some pcb tweaks (ordered this commit for rev 1)
Parts:
- U5: Digikey_PN AD5623RBRMZ-5REEL7CT-ND -> 505-AD5623RBRMZ-5-ND
- renumbered TP20 to TP1, TP21 to TP2, TP22 to TP3, TP11 to TP4, TP10 to TP5, TP9 to TP6
Changed lines of the file:
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@@
   (symbol (lib_id "Connector:TestPoint") (at 128.905 39.37 270) (unit 1)
     (in_bom yes) (on_board yes) (fields_autoplaced)
-    (property "Reference" "TP9" (id 0) (at 133.604 38.5353 90)
+    (property "Reference" "TP6" (id 0) (at 133.604 38.5353 90)
       (effects (font (size 1.27 1.27)) (justify left))
     )
@@
   (symbol (lib_id "Connector:TestPoint") (at 249.555 121.285 270) (unit 1)
     (in_bom yes) (on_board yes) (fields_autoplaced)
-    (property "Reference" "TP22" (id 0) (at 254.254 120.4503 90)
+    (property "Reference" "TP3" (id 0) (at 254.254 120.4503 90)
       (effects (font (size 1.27 1.27)) (justify left))
     )
@@
   (symbol (lib_id "Connector:TestPoint") (at 128.905 48.26 270) (unit 1)
     (in_bom yes) (on_board yes) (fields_autoplaced)
-    (property "Reference" "TP11" (id 0) (at 133.604 47.4253 90)
+    (property "Reference" "TP4" (id 0) (at 133.604 47.4253 90)
       (effects (font (size 1.27 1.27)) (justify left))
     )
@@
   (symbol (lib_id "Connector:TestPoint") (at 249.555 111.125 270) (unit 1)
     (in_bom yes) (on_board yes) (fields_autoplaced)
-    (property "Reference" "TP20" (id 0) (at 254.254 110.2903 90)
+    (property "Reference" "TP1" (id 0) (at 254.254 110.2903 90)
       (effects (font (size 1.27 1.27)) (justify left))
     )
@@
   (symbol (lib_id "Connector:TestPoint") (at 128.905 43.815 270) (unit 1)
     (in_bom yes) (on_board yes) (fields_autoplaced)
-    (property "Reference" "TP10" (id 0) (at 133.604 42.9803 90)
+    (property "Reference" "TP5" (id 0) (at 133.604 42.9803 90)
       (effects (font (size 1.27 1.27)) (justify left))
     )
@@
   (symbol (lib_id "Connector:TestPoint") (at 249.555 116.205 270) (unit 1)
     (in_bom yes) (on_board yes) (fields_autoplaced)
-    (property "Reference" "TP21" (id 0) (at 254.254 115.3703 90)
+    (property "Reference" "TP2" (id 0) (at 254.254 115.3703 90)
       (effects (font (size 1.27 1.27)) (justify left))
     )
@@
       (effects (font (size 1.27 1.27)) hide)
     )
-    (property "Digikey_PN" "AD5623RBRMZ-5REEL7CT-ND" (id 4) (at 144.145 139.065 0)
+    (property "Digikey_PN" "505-AD5623RBRMZ-5-ND" (id 4) (at 144.145 139.065 0)
       (effects (font (size 1.27 1.27)) hide)
     )
@@
       (reference "SW3") (unit 1) (value "BTN1") (footprint "Button_Switch_SMD:SW_SPST_TL3305A")
     )
+    (path "/901d513e-9a77-413a-906b-9d7eba70f2ee"
+      (reference "TP1") (unit 1) (value "Z Test") (footprint "TestPoint:TestPoint_Pad_D1.0mm")
+    )
+    (path "/f3d5151a-5cf4-4c7e-971f-107c6503f9a6"
+      (reference "TP2") (unit 1) (value "Y Test") (footprint "TestPoint:TestPoint_Pad_D1.0mm")
+    )
+    (path "/1ad85e5e-58e2-409a-b471-d18856edb5aa"
+      (reference "TP3") (unit 1) (value "X test") (footprint "TestPoint:TestPoint_Pad_D1.0mm")
+    )
+    (path "/5c6bf9e8-9d23-4b95-b376-ad423f1bfc33"
+      (reference "TP4") (unit 1) (value "ESP_GPIO16") (footprint "TestPoint:TestPoint_Pad_D1.0mm")
+    )
+    (path "/bdf21a19-4a3d-45c7-9ac1-306079e4836b"
+      (reference "TP5") (unit 1) (value "ESP_BOOT") (footprint "TestPoint:TestPoint_Pad_D1.0mm")
+    )
     (path "/16513962-623a-4494-912a-e58af61c3bdb"
-      (reference "TP9") (unit 1) (value "ESP_GPIO2") (footprint "TestPoint:TestPoint_Pad_D1.0mm")
-    )
-    (path "/bdf21a19-4a3d-45c7-9ac1-306079e4836b"
-      (reference "TP10") (unit 1) (value "ESP_BOOT") (footprint "TestPoint:TestPoint_Pad_D1.0mm")
-    )
-    (path "/5c6bf9e8-9d23-4b95-b376-ad423f1bfc33"
-      (reference "TP11") (unit 1) (value "ESP_GPIO16") (footprint "TestPoint:TestPoint_Pad_D1.0mm")
-    )
-    (path "/901d513e-9a77-413a-906b-9d7eba70f2ee"
-      (reference "TP20") (unit 1) (value "Z Test") (footprint "TestPoint:TestPoint_Pad_D1.0mm")
-    )
-    (path "/f3d5151a-5cf4-4c7e-971f-107c6503f9a6"
-      (reference "TP21") (unit 1) (value "Y Test") (footprint "TestPoint:TestPoint_Pad_D1.0mm")
-    )
-    (path "/1ad85e5e-58e2-409a-b471-d18856edb5aa"
-      (reference "TP22") (unit 1) (value "X test") (footprint "TestPoint:TestPoint_Pad_D1.0mm")
+      (reference "TP6") (unit 1) (value "ESP_GPIO2") (footprint "TestPoint:TestPoint_Pad_D1.0mm")
     )
     (path "/45d39a2f-8aab-473b-8561-f6bd933d6e5d"
